File: ampli.sch (KiCad schematic (older format))
At the start: 25 parts, among them J1 Conn_01x02, J2 Conn_01x02, Q1 stp16NF06

Commit message: modification Z input
Parts:
- R1: value 50R -> 100R
- R2: value 50RR_Small -> 100r
Changed lines of the file:
@@
 LIBS:power
 LIBS:Transistor_FET
+LIBS:ampli-cache
 EELAYER 25 0
 EELAYER END
@@
 P 1100 3800
 F 0 "R1" H 1130 3820 50  0000 L CNN
-F 1 "50R" H 1130 3760 50  0000 L CNN
+F 1 "100R" H 1130 3760 50  0000 L CNN
 F 2 "" H 1100 3800 50  0001 C CNN
 F 3 "" H 1100 3800 50  0001 C CNN
@@
 P 1400 3800
 F 0 "R2" H 1430 3820 50  0000 L CNN
-F 1 "50RR_Small" H 1430 3760 50  0000 L CNN
+F 1 "100r" H 1430 3760 50  0000 L CNN
 F 2 "" H 1400 3800 50  0001 C CNN
 F 3 "" H 1400 3800 50  0001 C CNN
